File: GPIB.sch (KiCad schematic (older format))
At the start: 20 parts

Commit message: ESP Serial interface
Parts:
- added D?: WIFI_CONNECTED_LED, symbol LED
- added R?: R, symbol R
- JP?: value JUMPER -> USB_LED_ENABLE
Connections:
- net GND: now also D?.2 (K)
- net GPIB_CTRL_DC: now also U?.26 (SPI2_SCK/I2S2_CK/I2C2_SCL/USART3_CTS/TIM1_CH1N/TSC_G6_IO3/PB13); no longer U?.21 (SPI2_SCK/I2C2_SCL/USART3_TX/CEC/TSC_SYNC/TIM2_CH3/PB10)
- net GPIB_CTRL_TE: now also U?.20 (TSC_G3_IO3/PB2); no longer U?.18 (TIM3_CH3/TIM1_CH2N/TSC_G3_IO2/EVENTOUT/USART3_CK18/ADC_IN8/PB0)
- net GPIB_DATA_TE: now also U?.18 (TIM3_CH3/TIM1_CH2N/TSC_G3_IO2/EVENTOUT/USART3_CK18/ADC_IN8/PB0); no longer U?.38 (SPI1_NSS/I2S1_WS/USART2_RX/USART4_RTS/TIM2_CH1_ETR/EVENTOUT/PA15)
- net at U?.15 (SRQ): now also U?.25 (TIM1_BKIN/TIM15_BKIN/SPI2_NSS/I2S2_WS/USART3_CK/TSC_G6_IO2/EVENTOUT/PB12); no longer U?.46 (SPI2_NSS/I2S2_WS/I2C1_SDA/IR_OUT/TIM17_CH1/EVENTOUT/CAN_TX/PB9)
- net at U?.16 (ATN): now also U?.46 (SPI2_NSS/I2S2_WS/I2C1_SDA/IR_OUT/TIM17_CH1/EVENTOUT/CAN_TX/PB9); no longer U?.45 (I2C1_SCL/CEC/TIM16_CH1/TSC_SYNC/CAN_RX/PB8)
- net at U?.17 (EOI): now also U?.45 (I2C1_SCL/CEC/TIM16_CH1/TSC_SYNC/CAN_RX/PB8); no longer U?.43 (I2C1_SDA/USART1_RX/USART4_CTS/TIM17_CH1N/TSC_G5_IO4/PB7)
- net at U?.18 (DAV): now also U?.43 (I2C1_SDA/USART1_RX/USART4_CTS/TIM17_CH1N/TSC_G5_IO4/PB7); no longer U?.42 (I2C1_SCL/USART1_TX/TIM16_CH1N/TSC_G5_I03/PB6)
- net at U?.19 (NRFD): now also U?.42 (I2C1_SCL/USART1_TX/TIM16_CH1N/TSC_G5_I03/PB6); no longer U?.41 (SPI1_MOSI/I2S1_SD/I2C1_SMBA/TIM16_BKIN/TIM3_CH2/WKUP6/PB5)
- net at U?.20 (NDAC): now also U?.41 (SPI1_MOSI/I2S1_SD/I2C1_SMBA/TIM16_BKIN/TIM3_CH2/WKUP6/PB5); no longer U?.40 (SPI1_MISO/I2S1_MCK/TIM17_BKIN/TIM3_CH1/TSC_G5_IO2/EVENTOUT/PB4)
- net at U?.21 (IFC): now also U?.40 (SPI1_MISO/I2S1_MCK/TIM17_BKIN/TIM3_CH1/TSC_G5_IO2/EVENTOUT/PB4); no longer U?.39 (SPI1_SCK/I2S1_CK/TIM2_CH2/TSC_G5_IO1/EVENTOUT/PB3)
- net at U?.22 (REN): now also U?.39 (SPI1_SCK/I2S1_CK/TIM2_CH2/TSC_G5_IO1/EVENTOUT/PB3); no longer U?.20 (TSC_G3_IO3/PB2)
- net ESP_SPI_CS/TXD2: now reaches U?.22 (USART3_RX/TIM2_CH4/EVENTOUT/TSC_G6_IO1/I2C2_SDA/PB11)
- new net: D?.1 (A), R?.1
- new net ESP_GPIO16: R?.2
- new net ESP_SPI_MISO/RXD2: U?.21 (SPI2_SCK/I2C2_SCL/USART3_TX/CEC/TSC_SYNC/TIM2_CH3/PB10)
Changed lines of the file:
@@
 U 1 1 55668641
 P 6550 1850
-F 0 "D?" H 6550 1950 50  0000 C CNN
-F 1 "GPIB_SEND" H 6550 1700 50  0000 C CNN
+F 0 "D?" H 6550 1750 50  0000 C CNN
+F 1 "GPIB_SEND" H 6550 1950 50  0000 C CNN
 F 2 "" H 6550 1850 60  0000 C CNN
 F 3 "" H 6550 1850 60  0000 C CNN
@@
 	1    0    0    -1
 $EndComp
-Text Notes 1800 6550 0    60   ~ 0
+Text Notes 2050 6400 0    60   ~ 0
 May replace this with lower\npin count in future versions
 $Comp
@@
 $EndComp
 Wire Wire Line
-	5250 4050 6000 4050
+	5250 4050 5950 4050
+Wire Wire Line
+	5950 4050 6000 4050
 Wire Wire Line
 	5250 3950 5400 3950
@@
 P 6550 1550
 F 0 "D?" H 6550 1650 50  0000 C CNN
-F 1 "USB ACTIVITY LED" H 6550 1450 50  0000 C CNN
+F 1 "USB ACTIVITY LED" H 6550 1400 50  0000 C CNN
 F 2 "" H 6550 1550 60  0000 C CNN
 F 3 "" H 6550 1550 60  0000 C CNN
@@
 	10650 1550 10750 1550
 Wire Wire Line
-	10750 1550 10750 1950
+	10750 1550 10750 1650
+Wire Wire Line
+	10750 1650 10750 1750
+Wire Wire Line
+	10750 1750 10750 1850
+Wire Wire Line
+	10750 1850 10750 1950
 Wire Wire Line
 	10650 1850 10750 1850
@@
 $EndComp
 Wire Wire Line
-	9300 1650 9300 1950
+	9300 1650 9300 1750
+Wire Wire Line
+	9300 1750 9300 1850
+Wire Wire Line
+	9300 1850 9300 1950
 Connection ~ 9300 1750
 Connection ~ 9300 1850
@@
 Connection ~ 1100 1450
 Wire Wire Line
-	1100 1450 1100 1700
+	1100 1450 1100 1550
+Wire Wire Line
+	1100 1550 1100 1700
 Wire Wire Line
 	1100 1700 1200 1700
@@
 Wire Wire Line
 	1300 3200 1850 3200
-Text HLabel 4000 7050 0    39   Input ~ 0
-ESP_SPI_CS
+Text HLabel 5500 5550 2    39   Input ~ 0
+ESP_SPI_CS/TXD2
 Text HLabel 4000 7150 0    39   Input ~ 0
 ESP_SPI_MOSI
-Text HLabel 4000 7250 0    39   Input ~ 0
-ESP_SPI_MISO
+Text HLabel 5500 5450 2    39   Input ~ 0
+ESP_SPI_MISO/RXD2
 Text HLabel 4000 7350 0    39   Input ~ 0
 ESP_SPI_CLK
-Text HLabel 4000 7450 0    39   Input ~ 0
-ESP_GPIO_16
 Text HLabel 4000 7550 0    39   Input ~ 0
 ESP_GPIO_4
@@
 	3400 2350 3400 2150
 Wire Wire Line
-	3400 2150 3850 2150
+	3400 2150 3550 2150
+Wire Wire Line
+	3550 2150 3600 2150
+Wire Wire Line
+	3600 2150 3850 2150
 Wire Wire Line
 	3600 2150 3600 2000
@@
 	5200 7050 5200 6950
 Wire Wire Line
-	5200 6950 5750 6950
+	5200 6950 5450 6950
+Wire Wire Line
+	5450 6950 5750 6950
 Connection ~ 5450 6950
 Wire Wire Line
-	5200 6550 5750 6550
+	5200 6550 5450 6550
+Wire Wire Line
+	5450 6550 5750 6550
 Connection ~ 5450 6550
 $Comp
@@
 	3400 6350 3400 6550
 Wire Wire Line
-	3400 6550 3850 6550
+	3400 6550 3550 6550
+Wire Wire Line
+	3550 6550 3600 6550
+Wire Wire Line
+	3600 6550 3850 6550
 Wire Wire Line
 	3600 6550 3600 6650
@@
 P 6300 4050
 F 0 "JP?" H 6300 4200 60  0000 C CNN
-F 1 "JUMPER" H 6300 3970 40  0000 C CNN
+F 1 "USB_LED_ENABLE" H 6300 3970 40  0000 C CNN
 F 2 "" H 6300 4050 60  0000 C CNN
 F 3 "" H 6300 4050 60  0000 C CNN
@@
 	6500 3800 7750 3800
 Wire Wire Line
-	7250 4650 7250 4850
+	7250 4750 7250 4850
 Wire Wire Line
 	7250 4850 7750 4850
 Wire Wire Line
-	7150 4750 7150 4950
-Wire Wire Line
-	7150 4950 7750 4950
-Wire Wire Line
-	7050 4850 7050 5050
+	7150 4850 7150 4950
 Wire Wire Line
 	7050 5050 7750 5050
 Wire Wire Line
-	6950 4950 6950 5150
-Wire Wire Line
 	6950 5150 7750 5150
 Wire Wire Line
-	6850 5050 6850 5250
-Wire Wire Line
 	6850 5250 7750 5250
 Wire Wire Line
-	6750 5150 6750 5350
-Wire Wire Line
 	6750 5350 7750 5350
 Wire Wire Line
-	6650 5250 6650 5450
-Wire Wire Line
 	6650 5450 7750 5450
 Wire Wire Line
-	6550 5350 6550 5550
-Wire Wire Line
-	6550 5550 7750 5550
-Wire Wire Line
-	5250 4450 5500 4450
+	6650 5550 7750 5550
 Wire Wire Line
 	5250 4550 5500 4550
-Text GLabel 5500 4450 2    39   Input ~ 0
-GPIB_CTRL_TE
+Wire Wire Line
+	5250 4650 5500 4650
 Text GLabel 5500 4550 2    39   Input ~ 0
 GPIB_CTRL_TE
-Wire Wire Line
-	5250 4650 7250 4650
-Wire Wire Line
-	5250 4750 7150 4750
-Wire Wire Line
-	5250 4850 7050 4850
-Wire Wire Line
-	5250 4950 6950 4950
-Wire Wire Line
-	5250 5050 6850 5050
-Wire Wire Line
-	5250 5150 6750 5150
-Wire Wire Line
-	5250 5250 6650 5250
-Wire Wire Line
-	5250 5350 6550 5350
-Wire Wire Line
-	5250 5450 5450 5450
-Text GLabel 5450 5450 2    39   Input ~ 0
+Text GLabel 5500 4650 2    39   Input ~ 0
+GPIB_CTRL_TE
+Wire Wire Line
+	5250 4750 7250 4750
+Wire Wire Line
+	5250 4850 7150 4850
+Wire Wire Line
+	5250 4950 7050 4950
+Wire Wire Line
+	5250 5050 6950 5050
+Wire Wire Line
+	5250 5150 6850 5150
+Wire Wire Line
+	5250 5250 6750 5250
+Wire Wire Line
+	5250 5350 6650 5350
+Text GLabel 5500 5750 2    39   Input ~ 0
 GPIB_CTRL_DC
 Wire Wire Line
@@
 Text GLabel 5400 3550 2    39   Input ~ 0
 GPIB_DATA_PE
-Wire Wire Line
-	5250 4250 5400 4250
-Text GLabel 5400 4250 2    39   Input ~ 0
+Text GLabel 5500 4450 2    39   Input ~ 0
 GPIB_DATA_TE
+Text HLabel 1050 1550 0    39   Input ~ 0
+ESP_RESET
+Wire Wire Line
+	1050 1550 1100 1550
+Connection ~ 1100 1550
+Wire Wire Line
+	5500 4450 5250 4450
+Wire Wire Line
+	7150 4950 7750 4950
+Wire Wire Line
+	7050 4950 7050 5050
+Wire Wire Line
+	6950 5050 6950 5150
+Wire Wire Line
+	6850 5150 6850 5250
+Wire Wire Line
+	6750 5250 6750 5350
+Wire Wire Line
+	6650 5350 6650 5450
+$Comp
+L LED D?
+U 1 1 556AE3D5
+P 6550 1200
+F 0 "D?" H 6550 1100 50  0000 C CNN
+F 1 "WIFI_CONNECTED_LED" H 6600 1300 50  0000 C CNN
+F 2 "" H 6550 1200 60  0000 C CNN
+F 3 "" H 6550 1200 60  0000 C CNN
+	1    6550 1200
+	1    0    0    -1
+$EndComp
+$Comp
+L R R?
+U 1 1 556AE4DE
+P 5950 1200
+F 0 "R?" V 6030 1200 40  0000 C CNN
+F 1 "R" V 5957 1201 40  0000 C CNN
+F 2 "" V 5880 1200 30  0000 C CNN
+F 3 "" H 5950 1200 30  0000 C CNN
+	1    5950 1200
+	0    1    1    0
+$EndComp
+$Comp
+L GND #PWR?
+U 1 1 556AE58B
+P 7200 1250
+F 0 "#PWR?" H 7200 1250 30  0001 C CNN
+F 1 "GND" H 7200 1180 30  0001 C CNN
+F 2 "" H 7200 1250 60  0000 C CNN
+F 3 "" H 7200 1250 60  0000 C CNN
+	1    7200 1250
+	1    0    0    -1
+$EndComp
+Wire Wire Line
+	5450 1200 5700 1200
+Wire Wire Line
+	6200 1200 6350 1200
+Wire Wire Line
+	6750 1200 7200 1200
+Wire Wire Line
+	7200 1200 7200 1250
+Text HLabel 5450 1200 0    39   Input ~ 0
+ESP_GPIO16
+Wire Wire Line
+	5250 5450 5500 5450
+Wire Wire Line
+	5250 5550 5500 5550
+Wire Wire Line
+	6650 5550 6650 5650
+Wire Wire Line
+	6650 5650 5250 5650
+Wire Wire Line
+	5250 5750 5500 5750
 $EndSCHEMATC
