File: power.sch (KiCad schematic (older format))
At the start: 16 parts

Commit message: Update main sch to reference heirarchy. Add some more stuff to ESP.
Parts:
- C? (x2): value 100u -> 47u
- C?: value C -> 47u
- R?: value R -> 270
Other:
- moved on the sheet: C?, CON?, D?, Q?, R?, U?, U?A, U?B

Commit message: Add testpoints and tidy up
Connections:
- net VBARREL renamed V_BARREL
Changed lines of the file:
@@
 LIBS:ap1117e50g-13
 LIBS:irlml2246tr
+LIBS:testpoint
 LIBS:Wifi-GPIB-cache
 EELAYER 25 0
@@
 Text Notes 7400 2750 0    60   ~ 0
 Unused
-Text HLabel 4800 2350 2    60   Input ~ 0
-VBARREL
-Text HLabel 4650 5250 0    60   Input ~ 0
-VBARREL
 $Comp
 L +5V #PWR?
@@
 Text Notes 2550 2950 0    60   ~ 0
 Must be greater than 6.6V\nLikely 12V max
+Text GLabel 4800 2350 2    60   Input ~ 0
+V_BARREL
+Text GLabel 4650 5250 0    60   Input ~ 0
+V_BARREL
 $EndSCHEMATC

Commit message: More cleanup and swap out M0 model
Parts:
- added W? (x2): TEST_GND, symbol TEST
- added W?: TEST_3.3V, symbol TEST
- added W?: TEST_VIN, symbol TEST
- added W?: TEST_5V, symbol TEST
Connections:
- net labels added: USB_D+, USB_D-, VCC, VIN
- net labels removed: V_BARREL
- wire segments 40 -> 50
Changed lines of the file:
@@
 LIBS:irlml2246tr
 LIBS:testpoint
+LIBS:vin
+LIBS:stm32f072cbt6
 LIBS:Wifi-GPIB-cache
 EELAYER 25 0
@@
 Text Notes 2550 2950 0    60   ~ 0
 Must be greater than 6.6V\nLikely 12V max
-Text GLabel 4800 2350 2    60   Input ~ 0
-V_BARREL
-Text GLabel 4650 5250 0    60   Input ~ 0
-V_BARREL
+Wire Wire Line
+	3700 4350 4100 4350
+Wire Wire Line
+	3700 4450 4100 4450
+Text HLabel 4100 4350 2    60   Input ~ 0
+USB_D-
+Text HLabel 4100 4450 2    60   Input ~ 0
+USB_D+
+$Comp
+L TEST W?
+U 1 1 55675FE3
+P 9850 3450
+F 0 "W?" H 9850 3510 40  0000 C CNN
+F 1 "TEST_GND" H 9850 3380 40  0000 C CNN
+F 2 "" H 9850 3450 60  0000 C CNN
+F 3 "" H 9850 3450 60  0000 C CNN
+	1    9850 3450
+	1    0    0    -1
+$EndComp
+$Comp
+L TEST W?
+U 1 1 55675FEA
+P 9850 3700
+F 0 "W?" H 9850 3760 40  0000 C CNN
+F 1 "TEST_GND" H 9850 3630 40  0000 C CNN
+F 2 "" H 9850 3700 60  0000 C CNN
+F 3 "" H 9850 3700 60  0000 C CNN
+	1    9850 3700
+	1    0    0    -1
+$EndComp
+$Comp
+L TEST W?
+U 1 1 55675FF1
+P 9850 3950
+F 0 "W?" H 9850 4010 40  0000 C CNN
+F 1 "TEST_3.3V" H 9850 3880 40  0000 C CNN
+F 2 "" H 9850 3950 60  0000 C CNN
+F 3 "" H 9850 3950 60  0000 C CNN
+	1    9850 3950
+	1    0    0    -1
+$EndComp
+$Comp
+L TEST W?
+U 1 1 55675FF8
+P 9850 4200
+F 0 "W?" H 9850 4260 40  0000 C CNN
+F 1 "TEST_VIN" H 9850 4130 40  0000 C CNN
+F 2 "" H 9850 4200 60  0000 C CNN
+F 3 "" H 9850 4200 60  0000 C CNN
+	1    9850 4200
+	1    0    0    -1
+$EndComp
+Wire Wire Line
+	9400 4200 9650 4200
+Wire Wire Line
+	9400 3950 9650 3950
+Wire Wire Line
+	9650 3700 9550 3700
+Wire Wire Line
+	9650 3450 9550 3450
+$Comp
+L TEST W?
+U 1 1 5567647D
+P 9850 4450
+F 0 "W?" H 9850 4510 40  0000 C CNN
+F 1 "TEST_5V" H 9850 4380 40  0000 C CNN
+F 2 "" H 9850 4450 60  0000 C CNN
+F 3 "" H 9850 4450 60  0000 C CNN
+	1    9850 4450
+	1    0    0    -1
+$EndComp
+Wire Wire Line
+	9400 4450 9650 4450
+$Comp
+L GND #PWR?
+U 1 1 5567667F
+P 9500 3500
+F 0 "#PWR?" H 9500 3500 30  0001 C CNN
+F 1 "GND" H 9500 3430 30  0001 C CNN
+F 2 "" H 9500 3500 60  0000 C CNN
+F 3 "" H 9500 3500 60  0000 C CNN
+	1    9500 3500
+	1    0    0    -1
+$EndComp
+$Comp
+L GND #PWR?
+U 1 1 556766BD
+P 9500 3750
+F 0 "#PWR?" H 9500 3750 30  0001 C CNN
+F 1 "GND" H 9500 3680 30  0001 C CNN
+F 2 "" H 9500 3750 60  0000 C CNN
+F 3 "" H 9500 3750 60  0000 C CNN
+	1    9500 3750
+	1    0    0    -1
+$EndComp
+$Comp
+L +3.3V #PWR?
+U 1 1 55676819
+P 9400 3900
+F 0 "#PWR?" H 9400 3860 30  0001 C CNN
+F 1 "+3.3V" H 9400 4010 30  0000 C CNN
+F 2 "" H 9400 3900 60  0000 C CNN
+F 3 "" H 9400 3900 60  0000 C CNN
+	1    9400 3900
+	1    0    0    -1
+$EndComp
+Wire Wire Line
+	9400 3950 9400 3900
+Wire Wire Line
+	9400 4450 9400 4400
+$Comp
+L +5V #PWR?
+U 1 1 556768F9
+P 9400 4400
+F 0 "#PWR?" H 9400 4490 20  0001 C CNN
+F 1 "+5V" H 9400 4490 30  0000 C CNN
+F 2 "" H 9400 4400 60  0000 C CNN
+F 3 "" H 9400 4400 60  0000 C CNN
+	1    9400 4400
+	1    0    0    -1
+$EndComp
+$Comp
+L PWR_FLAG #FLG?
+U 1 1 55676A42
+P 8700 3550
+F 0 "#FLG?" H 8700 3645 30  0001 C CNN
+F 1 "PWR_FLAG" H 8700 3730 30  0000 C CNN
+F 2 "" H 8700 3550 60  0000 C CNN
+F 3 "" H 8700 3550 60  0000 C CNN
+	1    8700 3550
+	1    0    0    -1
+$EndComp
+$Comp
+L VCC #PWR?
+U 1 1 55676BEC
+P 8950 3450
+F 0 "#PWR?" H 8950 3550 30  0001 C CNN
+F 1 "VCC" H 8950 3550 30  0000 C CNN
+F 2 "" H 8950 3450 60  0000 C CNN
+F 3 "" H 8950 3450 60  0000 C CNN
+	1    8950 3450
+	1    0    0    -1
+$EndComp
+$Comp
+L VIN #PWR?
+U 1 1 55676D63
+P 9400 4150
+F 0 "#PWR?" H 9400 4250 30  0001 C CNN
+F 1 "VIN" H 9400 4250 30  0000 C CNN
+F 2 "" H 9400 4150 60  0000 C CNN
+F 3 "" H 9400 4150 60  0000 C CNN
+	1    9400 4150
+	1    0    0    -1
+$EndComp
+Wire Wire Line
+	9400 4200 9400 4150
+$Comp
+L VIN #PWR?
+U 1 1 5567710F
+P 4800 2350
+F 0 "#PWR?" H 4800 2450 30  0001 C CNN
+F 1 "VIN" H 4800 2450 30  0000 C CNN
+F 2 "" H 4800 2350 60  0000 C CNN
+F 3 "" H 4800 2350 60  0000 C CNN
+	1    4800 2350
+	1    0    0    -1
+$EndComp
+$Comp
+L VIN #PWR?
+U 1 1 556772F1
+P 4650 5250
+F 0 "#PWR?" H 4650 5350 30  0001 C CNN
+F 1 "VIN" H 4650 5350 30  0000 C CNN
+F 2 "" H 4650 5250 60  0000 C CNN
+F 3 "" H 4650 5250 60  0000 C CNN
+	1    4650 5250
+	1    0    0    -1
+$EndComp
 $EndSCHEMATC

Commit message: Finish USB and test points for power
Parts:
- added R?: 100k, symbol R
Connections:
- net labels removed: VCC
- wire segments 50 -> 64
Other:
- note added: "Ideally also add shield (with RC to GND)"
- note added: "Need to add ESD protection here.\nTermination resistors provided internally in STM32."
- moved on the sheet: W?
Changed lines of the file:
@@
 LIBS:vin
 LIBS:stm32f072cbt6
+LIBS:nuf2221w1
 LIBS:Wifi-GPIB-cache
 EELAYER 25 0
@@
 	3800 2550 3950 2550
 Wire Wire Line
-	3950 2450 3950 2850
+	3950 2450 3950 2550
+Wire Wire Line
+	3950 2550 3950 2850
 Wire Wire Line
 	3800 2450 3950 2450
@@
 	4250 2850 4250 3000
 Wire Wire Line
-	4250 3000 5200 3000
+	4250 3000 4650 3000
+Wire Wire Line
+	4650 3000 5200 3000
 Wire Wire Line
 	4650 3000 4650 3050
 Wire Wire Line
-	4250 3500 4250 3700
+	4250 3500 4250 3550
+Wire Wire Line
+	4250 3550 4250 3700
 Wire Wire Line
 	4250 3550 4650 3550
@@
 	6700 3100 6700 3950
 Wire Wire Line
-	3700 4250 6450 4250
-Wire Wire Line
 	6850 4250 8050 4250
 Wire Wire Line
@@
 	7500 2950 7250 2950
 Wire Wire Line
-	7250 2950 7250 3400
+	7250 2950 7250 3150
+Wire Wire Line
+	7250 3150 7250 3400
 Wire Wire Line
 	7500 3150 7250 3150
 Connection ~ 7250 3150
 Wire Wire Line
-	4650 5250 5000 5250
+	4650 5250 4850 5250
+Wire Wire Line
+	4850 5250 5000 5250
 Wire Wire Line
 	6900 5150 6900 5250
 Wire Wire Line
-	6900 5250 7200 5250
+	6900 5250 7050 5250
+Wire Wire Line
+	7050 5250 7200 5250
 Wire Wire Line
 	7600 5550 7600 5650
 Wire Wire Line
-	8000 5250 8500 5250
+	8000 5250 8350 5250
+Wire Wire Line
+	8350 5250 8500 5250
 Wire Wire Line
 	8500 5250 8500 5100
 Wire Wire Line
-	5800 5250 6250 5250
+	5800 5250 6050 5250
+Wire Wire Line
+	6050 5250 6250 5250
 Wire Wire Line
 	6250 5250 6250 5150
@@
 	5400 5550 5400 5650
 Wire Wire Line
-	3800 2350 4800 2350
+	3800 2350 4250 2350
+Wire Wire Line
+	4250 2350 4550 2350
+Wire Wire Line
+	4550 2350 4800 2350
 Connection ~ 4550 2350
 $Comp
@@
 Must be greater than 6.6V\nLikely 12V max
 Wire Wire Line
-	3700 4350 4100 4350
-Wire Wire Line
-	3700 4450 4100 4450
-Text HLabel 4100 4350 2    60   Input ~ 0
+	3700 4350 5600 4350
+Wire Wire Line
+	3700 4450 5600 4450
+Text HLabel 5600 4350 2    60   Input ~ 0
 USB_D-
-Text HLabel 4100 4450 2    60   Input ~ 0
+Text HLabel 5600 4450 2    60   Input ~ 0
 USB_D+
 $Comp
 L TEST W?
 U 1 1 55675FE3
-P 9850 3450
-F 0 "W?" H 9850 3510 40  0000 C CNN
-F 1 "TEST_GND" H 9850 3380 40  0000 C CNN
-F 2 "" H 9850 3450 60  0000 C CNN
-F 3 "" H 9850 3450 60  0000 C CNN
-	1    9850 3450
+P 9850 4700
+F 0 "W?" H 9850 4760 40  0000 C CNN
+F 1 "TEST_GND" H 9850 4630 40  0000 C CNN
+F 2 "" H 9850 4700 60  0000 C CNN
+F 3 "" H 9850 4700 60  0000 C CNN
+	1    9850 4700
 	1    0    0    -1
 $EndComp
@@
 L TEST W?
 U 1 1 55675FEA
-P 9850 3700
-F 0 "W?" H 9850 3760 40  0000 C CNN
-F 1 "TEST_GND" H 9850 3630 40  0000 C CNN
-F 2 "" H 9850 3700 60  0000 C CNN
-F 3 "" H 9850 3700 60  0000 C CNN
-	1    9850 3700
+P 9850 4950
+F 0 "W?" H 9850 5010 40  0000 C CNN
+F 1 "TEST_GND" H 9850 4880 40  0000 C CNN
+F 2 "" H 9850 4950 60  0000 C CNN
+F 3 "" H 9850 4950 60  0000 C CNN
+	1    9850 4950
 	1    0    0    -1
 $EndComp
@@
 $EndComp
 Wire Wire Line
-	9400 4200 9650 4200
-Wire Wire Line
-	9400 3950 9650 3950
-Wire Wire Line
-	9650 3700 9550 3700
-Wire Wire Line
-	9650 3450 9550 3450
+	9500 4200 9650 4200
+Wire Wire Line
+	9500 3950 9650 3950
+Wire Wire Line
+	9500 4950 9650 4950
+Wire Wire Line
+	9500 4700 9650 4700
 $Comp
 L TEST W?
@@
 $EndComp
 Wire Wire Line
-	9400 4450 9650 4450
+	9500 4450 9650 4450
 $Comp
 L GND #PWR?
 U 1 1 5567667F
-P 9500 3500
-F 0 "#PWR?" H 9500 3500 30  0001 C CNN
-F 1 "GND" H 9500 3430 30  0001 C CNN
-F 2 "" H 9500 3500 60  0000 C CNN
-F 3 "" H 9500 3500 60  0000 C CNN
-	1    9500 3500
+P 9500 4750
+F 0 "#PWR?" H 9500 4750 30  0001 C CNN
+F 1 "GND" H 9500 4680 30  0001 C CNN
+F 2 "" H 9500 4750 60  0000 C CNN
+F 3 "" H 9500 4750 60  0000 C CNN
+	1    9500 4750
 	1    0    0    -1
 $EndComp
@@
 L GND #PWR?
 U 1 1 556766BD
-P 9500 3750
-F 0 "#PWR?" H 9500 3750 30  0001 C CNN
-F 1 "GND" H 9500 3680 30  0001 C CNN
-F 2 "" H 9500 3750 60  0000 C CNN
-F 3 "" H 9500 3750 60  0000 C CNN
-	1    9500 3750
+P 9500 5000
+F 0 "#PWR?" H 9500 5000 30  0001 C CNN
+F 1 "GND" H 9500 4930 30  0001 C CNN
+F 2 "" H 9500 5000 60  0000 C CNN
+F 3 "" H 9500 5000 60  0000 C CNN
+	1    9500 5000
 	1    0    0    -1
 $EndComp
@@
 L +3.3V #PWR?
 U 1 1 55676819
-P 9400 3900
-F 0 "#PWR?" H 9400 3860 30  0001 C CNN
-F 1 "+3.3V" H 9400 4010 30  0000 C CNN
-F 2 "" H 9400 3900 60  0000 C CNN
-F 3 "" H 9400 3900 60  0000 C CNN
-	1    9400 3900
-	1    0    0    -1
-$EndComp
-Wire Wire Line
-	9400 3950 9400 3900
-Wire Wire Line
-	9400 4450 9400 4400
+P 9500 3900
+F 0 "#PWR?" H 9500 3860 30  0001 C CNN
+F 1 "+3.3V" H 9500 4010 30  0000 C CNN
+F 2 "" H 9500 3900 60  0000 C CNN
+F 3 "" H 9500 3900 60  0000 C CNN
+	1    9500 3900
+	1    0    0    -1
+$EndComp
+Wire Wire Line
+	9500 3950 9500 3900
+Wire Wire Line
+	9500 4450 9500 4400
 $Comp
 L +5V #PWR?
 U 1 1 556768F9
-P 9400 4400
-F 0 "#PWR?" H 9400 4490 20  0001 C CNN
-F 1 "+5V" H 9400 4490 30  0000 C CNN
-F 2 "" H 9400 4400 60  0000 C CNN
-F 3 "" H 9400 4400 60  0000 C CNN
-	1    9400 4400
-	1    0    0    -1
-$EndComp
-$Comp
-L PWR_FLAG #FLG?
-U 1 1 55676A42
-P 8700 3550
-F 0 "#FLG?" H 8700 3645 30  0001 C CNN
-F 1 "PWR_FLAG" H 8700 3730 30  0000 C CNN
-F 2 "" H 8700 3550 60  0000 C CNN
-F 3 "" H 8700 3550 60  0000 C CNN
-	1    8700 3550
-	1    0    0    -1
-$EndComp
-$Comp
-L VCC #PWR?
-U 1 1 55676BEC
-P 8950 3450
-F 0 "#PWR?" H 8950 3550 30  0001 C CNN
-F 1 "VCC" H 8950 3550 30  0000 C CNN
-F 2 "" H 8950 3450 60  0000 C CNN
-F 3 "" H 8950 3450 60  0000 C CNN
-	1    8950 3450
+P 9500 4400
+F 0 "#PWR?" H 9500 4490 20  0001 C CNN
+F 1 "+5V" H 9500 4490 30  0000 C CNN
+F 2 "" H 9500 4400 60  0000 C CNN
+F 3 "" H 9500 4400 60  0000 C CNN
+	1    9500 4400
 	1    0    0    -1
 $EndComp
@@
 L VIN #PWR?
 U 1 1 55676D63
-P 9400 4150
-F 0 "#PWR?" H 9400 4250 30  0001 C CNN
-F 1 "VIN" H 9400 4250 30  0000 C CNN
-F 2 "" H 9400 4150 60  0000 C CNN
-F 3 "" H 9400 4150 60  0000 C CNN
-	1    9400 4150
-	1    0    0    -1
-$EndComp
-Wire Wire Line
-	9400 4200 9400 4150
+P 9500 4150
+F 0 "#PWR?" H 9500 4250 30  0001 C CNN
+F 1 "VIN" H 9500 4250 30  0000 C CNN
+F 2 "" H 9500 4150 60  0000 C CNN
+F 3 "" H 9500 4150 60  0000 C CNN
+	1    9500 4150
+	1    0    0    -1
+$EndComp
+Wire Wire Line
+	9500 4200 9500 4150
 $Comp
 L VIN #PWR?
@@
 	1    0    0    -1
 $EndComp
+Wire Wire Line
+	6450 4250 3700 4250
+Wire Wire Line
+	3700 4550 4300 4550
+Wire Wire Line
+	4300 4550 4300 4600
+$Comp
+L R R?
+U 1 1 55678D89
+P 4300 4850
+F 0 "R?" V 4380 4850 40  0000 C CNN
+F 1 "100k" V 4307 4851 40  0000 C CNN
+F 2 "" V 4230 4850 30  0000 C CNN
+F 3 "" H 4300 4850 30  0000 C CNN
+	1    4300 4850
+	1    0    0    -1
+$EndComp
+$Comp
+L GND #PWR?
+U 1 1 55678E06
+P 4300 5100
+F 0 "#PWR?" H 4300 5100 30  0001 C CNN
+F 1 "GND" H 4300 5030 30  0001 C CNN
+F 2 "" H 4300 5100 60  0000 C CNN
+F 3 "" H 4300 5100 60  0000 C CNN
+	1    4300 5100
+	1    0    0    -1
+$EndComp
+Wire Wire Line
+	9500 4700 9500 4750
+Wire Wire Line
+	9500 4950 9500 5000
+Text Notes 3950 4200 0    60   ~ 0
+Need to add ESD protection here.\nTermination resistors provided internally in STM32.
+Text Notes 4350 4600 0    60   ~ 0
+Ideally also add shield (with RC to GND)
 $EndSCHEMATC

Commit message: Think sch finished
Parts:
- added TP?: TESTPOINT, symbol TESTPOINT
Connections:
- net at C?.1, R?.1, R?.2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: now also TP?.1
Changed lines of the file:
@@
 $EndComp
 $Comp
-L +5V #PWR?
+L +5V #PWR01
 U 1 1 55661F39
 P 5600 2600
-F 0 "#PWR?" H 5600 2690 20  0001 C CNN
+F 0 "#PWR01" H 5600 2690 20  0001 C CNN
 F 1 "+5V" H 5600 2690 30  0000 C CNN
 F 2 "" H 5600 2600 60  0000 C CNN
@@
 $EndComp
 $Comp
-L GND #PWR?
+L GND #PWR02
 U 1 1 55661F58
 P 5600 3600
-F 0 "#PWR?" H 5600 3600 30  0001 C CNN
+F 0 "#PWR02" H 5600 3600 30  0001 C CNN
 F 1 "GND" H 5600 3530 30  0001 C CNN
 F 2 "" H 5600 3600 60  0000 C CNN
@@
 $EndComp
 $Comp
-L GND #PWR?
+L GND #PWR03
 U 1 1 556622F1
 P 3950 2850
-F 0 "#PWR?" H 3950 2850 30  0001 C CNN
+F 0 "#PWR03" H 3950 2850 30  0001 C CNN
 F 1 "GND" H 3950 2780 30  0001 C CNN
 F 2 "" H 3950 2850 60  0000 C CNN
@@
 $EndComp
 $Comp
-L GND #PWR?
+L GND #PWR04
 U 1 1 5566238D
 P 4250 3700
-F 0 "#PWR?" H 4250 3700 30  0001 C CNN
+F 0 "#PWR04" H 4250 3700 30  0001 C CNN
 F 1 "GND" H 4250 3630 30  0001 C CNN
 F 2 "" H 4250 3700 60  0000 C CNN
@@
 $EndComp
 $Comp
-L +3.3V #PWR?
+L +3.3V #PWR05
 U 1 1 556626E8
 P 5000 3200
-F 0 "#PWR?" H 5000 3160 30  0001 C CNN
+F 0 "#PWR05" H 5000 3160 30  0001 C CNN
 F 1 "+3.3V" H 5000 3310 30  0000 C CNN
 F 2 "" H 5000 3200 60  0000 C CNN
@@
 $EndComp
 $Comp
-L +5V #PWR?
+L +5V #PWR06
 U 1 1 55662D5C
 P 8050 4250
-F 0 "#PWR?" H 8050 4340 20  0001 C CNN
+F 0 "#PWR06" H 8050 4340 20  0001 C CNN
 F 1 "+5V" H 8050 4340 30  0000 C CNN
 F 2 "" H 8050 4250 60  0000 C CNN
@@
 $EndComp
 $Comp
-L +5V #PWR?
+L +5V #PWR07
 U 1 1 5566302B
 P 6150 1850
-F 0 "#PWR?" H 6150 1940 20  0001 C CNN
+F 0 "#PWR07" H 6150 1940 20  0001 C CNN
 F 1 "+5V" H 6150 1940 30  0000 C CNN
 F 2 "" H 6150 1850 60  0000 C CNN
@@
 $EndComp
 $Comp
-L GND #PWR?
+L GND #PWR08
 U 1 1 5566304B
 P 7600 1850
-F 0 "#PWR?" H 7600 1850 30  0001 C CNN
+F 0 "#PWR08" H 7600 1850 30  0001 C CNN
 F 1 "GND" H 7600 1780 30  0001 C CNN
 F 2 "" H 7600 1850 60  0000 C CNN
@@
 $EndComp
 $Comp
-L GND #PWR?
+L GND #PWR09
 U 1 1 55663314
 P 3900 4900
-F 0 "#PWR?" H 3900 4900 30  0001 C CNN
+F 0 "#PWR09" H 3900 4900 30  0001 C CNN
 F 1 "GND" H 3900 4830 30  0001 C CNN
 F 2 "" H 3900 4900 60  0000 C CNN
@@
 $EndComp
 $Comp
-L GND #PWR?
+L GND #PWR010
 U 1 1 556634C1
 P 7250 3400
-F 0 "#PWR?" H 7250 3400 30  0001 C CNN
+F 0 "#PWR010" H 7250 3400 30  0001 C CNN
 F 1 "GND" H 7250 3330 30  0001 C CNN
 F 2 "" H 7250 3400 60  0000 C CNN
@@
 Unused
 $Comp
-L +5V #PWR?
+L +5V #PWR011
 U 1 1 55663FD0
 P 6900 5150
-F 0 "#PWR?" H 6900 5240 20  0001 C CNN
+F 0 "#PWR011" H 6900 5240 20  0001 C CNN
 F 1 "+5V" H 6900 5240 30  0000 C CNN
 F 2 "" H 6900 5150 60  0000 C CNN
@@
 $EndComp
 $Comp
-L GND #PWR?
+L GND #PWR012
 U 1 1 5566404D
 P 7600 5650
-F 0 "#PWR?" H 7600 5650 30  0001 C CNN
+F 0 "#PWR012" H 7600 5650 30  0001 C CNN
 F 1 "GND" H 7600 5580 30  0001 C CNN
 F 2 "" H 7600 5650 60  0000 C CNN
@@
 $EndComp
 $Comp
-L +3.3V #PWR?
+L +3.3V #PWR013
 U 1 1 5566409E
 P 8500 5100
-F 0 "#PWR?" H 8500 5060 30  0001 C CNN
+F 0 "#PWR013" H 8500 5060 30  0001 C CNN
 F 1 "+3.3V" H 8500 5210 30  0000 C CNN
 F 2 "" H 8500 5100 60  0000 C CNN
@@
 $EndComp
 $Comp
-L +5V #PWR?
+L +5V #PWR014
 U 1 1 55664199
 P 6250 5150
-F 0 "#PWR?" H 6250 5240 20  0001 C CNN
+F 0 "#PWR014" H 6250 5240 20  0001 C CNN
 F 1 "+5V" H 6250 5240 30  0000 C CNN
 F 2 "" H 6250 5150 60  0000 C CNN
@@
 $EndComp
 $Comp
-L GND #PWR?
+L GND #PWR015
 U 1 1 55664236
 P 5400 5650
-F 0 "#PWR?" H 5400 5650 30  0001 C CNN
+F 0 "#PWR015" H 5400 5650 30  0001 C CNN
 F 1 "GND" H 5400 5580 30  0001 C CNN
 F 2 "" H 5400 5650 60  0000 C CNN
@@
 	3800 2550 3950 2550
 Wire Wire Line
-	3950 2450 3950 2550
-Wire Wire Line
-	3950 2550 3950 2850
+	3950 2450 3950 2850
 Wire Wire Line
 	3800 2450 3950 2450
@@
 	4250 2850 4250 3000
 Wire Wire Line
-	4250 3000 4650 3000
-Wire Wire Line
-	4650 3000 5200 3000
-Wire Wire Line
-	4650 3000 4650 3050
-Wire Wire Line
-	4250 3500 4250 3550
-Wire Wire Line
-	4250 3550 4250 3700
+	4250 3000 5200 3000
+Wire Wire Line
+	4650 2850 4650 3050
+Wire Wire Line
+	4250 3500 4250 3700
 Wire Wire Line
 	4250 3550 4650 3550
@@
 	7500 2950 7250 2950
 Wire Wire Line
-	7250 2950 7250 3150
-Wire Wire Line
-	7250 3150 7250 3400
+	7250 2950 7250 3400
 Wire Wire Line
 	7500 3150 7250 3150
 Connection ~ 7250 3150
 Wire Wire Line
-	4650 5250 4850 5250
-Wire Wire Line
-	4850 5250 5000 5250
+	4650 5250 5000 5250
 Wire Wire Line
 	6900 5150 6900 5250
 Wire Wire Line
-	6900 5250 7050 5250
-Wire Wire Line
-	7050 5250 7200 5250
+	6900 5250 7200 5250
 Wire Wire Line
 	7600 5550 7600 5650
 Wire Wire Line
-	8000 5250 8350 5250
-Wire Wire Line
-	8350 5250 8500 5250
+	8000 5250 8500 5250
 Wire Wire Line
 	8500 5250 8500 5100
 Wire Wire Line
-	5800 5250 6050 5250
-Wire Wire Line
-	6050 5250 6250 5250
+	5800 5250 6250 5250
 Wire Wire Line
 	6250 5250 6250 5150
@@
 	5400 5550 5400 5650
 Wire Wire Line
-	3800 2350 4250 2350
-Wire Wire Line
-	4250 2350 4550 2350
-Wire Wire Line
-	4550 2350 4800 2350
+	3800 2350 4800 2350
 Connection ~ 4550 2350
 $Comp
-L GND #PWR?
+L GND #PWR016
 U 1 1 5566547F
 P 4850 5800
-F 0 "#PWR?" H 4850 5800 30  0001 C CNN
+F 0 "#PWR016" H 4850 5800 30  0001 C CNN
 F 1 "GND" H 4850 5730 30  0001 C CNN
 F 2 "" H 4850 5800 60  0000 C CNN
@@
 Connection ~ 6050 5250
 $Comp
-L GND #PWR?
+L GND #PWR017
 U 1 1 55665981
 P 6050 5800
-F 0 "#PWR?" H 6050 5800 30  0001 C CNN
+F 0 "#PWR017" H 6050 5800 30  0001 C CNN
 F 1 "GND" H 6050 5730 30  0001 C CNN
 F 2 "" H 6050 5800 60  0000 C CNN
@@
 Connection ~ 8350 5250
 $Comp
-L GND #PWR?
+L GND #PWR018
 U 1 1 55665BA8
 P 8350 5900
-F 0 "#PWR?" H 8350 5900 30  0001 C CNN
+F 0 "#PWR018" H 8350 5900 30  0001 C CNN
 F 1 "GND" H 8350 5830 30  0001 C CNN
 F 2 "" H 8350 5900 60  0000 C CNN
@@
 Connection ~ 7050 5250
 $Comp
-L GND #PWR?
+L GND #PWR019
 U 1 1 55665CA1
 P 7050 5900
-F 0 "#PWR?" H 7050 5900 30  0001 C CNN
+F 0 "#PWR019" H 7050 5900 30  0001 C CNN
 F 1 "GND" H 7050 5830 30  0001 C CNN
 F 2 "" H 7050 5900 60  0000 C CNN
@@
 	9500 4450 9650 4450
 $Comp
-L GND #PWR?
+L GND #PWR020
 U 1 1 5567667F
 P 9500 4750
-F 0 "#PWR?" H 9500 4750 30  0001 C CNN
+F 0 "#PWR020" H 9500 4750 30  0001 C CNN
 F 1 "GND" H 9500 4680 30  0001 C CNN
 F 2 "" H 9500 4750 60  0000 C CNN
@@
 $EndComp
 $Comp
-L GND #PWR?
+L GND #PWR021
 U 1 1 556766BD
 P 9500 5000
-F 0 "#PWR?" H 9500 5000 30  0001 C CNN
+F 0 "#PWR021" H 9500 5000 30  0001 C CNN
 F 1 "GND" H 9500 4930 30  0001 C CNN
 F 2 "" H 9500 5000 60  0000 C CNN
@@
 $EndComp
 $Comp
-L +3.3V #PWR?
+L +3.3V #PWR022
 U 1 1 55676819
 P 9500 3900
-F 0 "#PWR?" H 9500 3860 30  0001 C CNN
+F 0 "#PWR022" H 9500 3860 30  0001 C CNN
 F 1 "+3.3V" H 9500 4010 30  0000 C CNN
 F 2 "" H 9500 3900 60  0000 C CNN
@@
 	9500 4450 9500 4400
 $Comp
-L +5V #PWR?
+L +5V #PWR023
 U 1 1 556768F9
 P 9500 4400
-F 0 "#PWR?" H 9500 4490 20  0001 C CNN
+F 0 "#PWR023" H 9500 4490 20  0001 C CNN
 F 1 "+5V" H 9500 4490 30  0000 C CNN
 F 2 "" H 9500 4400 60  0000 C CNN
@@
 $EndComp
 $Comp
-L VIN #PWR?
+L VIN #PWR024
 U 1 1 55676D63
 P 9500 4150
-F 0 "#PWR?" H 9500 4250 30  0001 C CNN
+F 0 "#PWR024" H 9500 4250 30  0001 C CNN
 F 1 "VIN" H 9500 4250 30  0000 C CNN
 F 2 "" H 9500 4150 60  0000 C CNN
@@
 	9500 4200 9500 4150
 $Comp
-L VIN #PWR?
+L VIN #PWR025
 U 1 1 5567710F
 P 4800 2350
-F 0 "#PWR?" H 4800 2450 30  0001 C CNN
+F 0 "#PWR025" H 4800 2450 30  0001 C CNN
 F 1 "VIN" H 4800 2450 30  0000 C CNN
 F 2 "" H 4800 2350 60  0000 C CNN
@@
 $EndComp
 $Comp
-L VIN #PWR?
+L VIN #PWR026
 U 1 1 556772F1
 P 4650 5250
-F 0 "#PWR?" H 4650 5350 30  0001 C CNN
+F 0 "#PWR026" H 4650 5350 30  0001 C CNN
 F 1 "VIN" H 4650 5350 30  0000 C CNN
 F 2 "" H 4650 5250 60  0000 C CNN
@@
 $EndComp
 $Comp
-L GND #PWR?
+L GND #PWR027
 U 1 1 55678E06
 P 4300 5100
-F 0 "#PWR?" H 4300 5100 30  0001 C CNN
+F 0 "#PWR027" H 4300 5100 30  0001 C CNN
 F 1 "GND" H 4300 5030 30  0001 C CNN
 F 2 "" H 4300 5100 60  0000 C CNN
@@
 Text Notes 4350 4600 0    60   ~ 0
 Ideally also add shield (with RC to GND)
+$Comp
+L TESTPOINT TP?
+U 1 1 556C2967
+P 4650 2850
+F 0 "TP?" H 4650 3100 60  0000 C CNN
+F 1 "TESTPOINT" H 4650 2800 60  0001 C CNN
+F 2 "" H 4650 2850 60  0000 C CNN
+F 3 "" H 4650 2850 60  0000 C CNN
+	1    4650 2850
+	1    0    0    -1
+$EndComp
 $EndSCHEMATC
