File: power.sch (KiCad schematic (older format))
At the start: 22 parts, among them CON1 POWER_BARREL, Q1 IRLML2246TR, U1 MICRO-B_USB, U2 AP1117E50G-13, U3 LM358, U4 BA33BC0FP-E2

Commit message: Remove Barrel Jack and associated power circuits. Unnecessary for now and add a lot of complexity / BOM cost
Parts:
- removed C1: 100n, Capacitors_SMD:C_0603_HandSoldering, symbol C
- removed C2, C3: 47u, Capacitors_SMD:c_elec_8x6.5, symbol C
- removed CON1: POWER_BARREL, Connect:BARREL_JACK, symbol BARREL_JACK
- removed Q1: IRLML2246TR, SOT23_Transistor_RevA_03Aug2010:SOT23_Transistor_Handsoldering_RevA_03Aug2010, symbol IRLML2246TR
- removed R1, R2: 10K, Resistors_SMD:R_0603_HandSoldering, symbol R
- removed TP1: TESTPOINT, Connect:PINTST, symbol TESTPOINT
- removed TP12: TESTPOINT, Connect:TESTPOINT, symbol TESTPOINT
- removed U2: AP1117E50G-13, SOT223:SOT223, symbol AP1117E50G-13
- removed U3: LM358, Housings_SOIC:SOIC-8-1EP_3.9x4.9mm_Pitch1.27mm, symbol LM358
- D1: value LED_POWER -> PWR
Connections:
- net +5V: now also U1.1 (VBUS)
Other:
- note removed: "Must be greater than 6.6V\nLikely 12V max"
- note removed: "Power Circuits."
- note removed: "Switches between USB and barrel jack,\nalways preferring barrel jack if available.\nPrevents reverse current being driven\nover USB. Provides Reverse polarity \nprotection."
- note removed: "Unused"
