File: Wifi.sch (KiCad schematic (older format))
At the start: 15 parts, among them P5 CONN_4, U8 ESP-12/07v2/08v2

Commit message: Start routing
Parts:
- C12: footprint (none) -> Capacitors_SMD:C_0603_HandSoldering
- JP2: footprint (none) -> Pin_Headers:Pin_Header_Straight_1x02
- P5: footprint (none) -> Pin_Headers:Pin_Header_Straight_1x04
- R10, R11: footprint (none) -> Resistors_SMD:R_0603_HandSoldering
- TP10, TP2, TP3, TP4, TP5, TP6, TP7, TP8, TP9: footprint (none) -> Connect:PINTST
- U8: footprint (none) -> ESP8266:ESP-07
Changed lines of the file:
@@
 F 0 "U8" H 6050 4800 60  0000 C CNN
 F 1 "ESP-12/07v2/08v2" H 6050 3700 60  0000 C CNN
-F 2 "" H 6050 4250 60  0000 C CNN
+F 2 "ESP8266:ESP-07" H 6050 4250 60  0001 C CNN
 F 3 "" H 6050 4250 60  0000 C CNN
 	1    6050 4250
@@
 F 0 "P5" V 6750 2350 50  0000 C CNN
 F 1 "CONN_4" V 6850 2350 50  0000 C CNN
-F 2 "" H 6800 2350 60  0000 C CNN
+F 2 "Pin_Headers:Pin_Header_Straight_1x04" H 6800 2350 60  0001 C CNN
 F 3 "" H 6800 2350 60  0000 C CNN
 	1    6800 2350
@@
 $EndComp
 $Comp
-L GND #PWR056
+L GND #PWR60
 U 1 1 55667722
 P 6650 2900
-F 0 "#PWR056" H 6650 2900 30  0001 C CNN
+F 0 "#PWR60" H 6650 2900 30  0001 C CNN
 F 1 "GND" H 6650 2830 30  0001 C CNN
 F 2 "" H 6650 2900 60  0000 C CNN
@@
 $EndComp
 $Comp
-L +3.3V #PWR057
+L +3.3V #PWR59
 U 1 1 55667729
 P 6400 2950
-F 0 "#PWR057" H 6400 2910 30  0001 C CNN
+F 0 "#PWR59" H 6400 2910 30  0001 C CNN
 F 1 "+3.3V" H 6400 3060 30  0000 C CNN
 F 2 "" H 6400 2950 60  0000 C CNN
@@
 F 0 "JP2" H 5600 3050 60  0000 C CNN
 F 1 "ESP_FLASH_JUMP" H 5600 2820 40  0000 C CNN
-F 2 "" H 5600 2900 60  0000 C CNN
+F 2 "Pin_Headers:Pin_Header_Straight_1x02" H 5600 2900 60  0001 C CNN
 F 3 "" H 5600 2900 60  0000 C CNN
 	1    5600 2900
@@
 F 0 "R10" V 5130 2650 40  0000 C CNN
 F 1 "R" V 5057 2651 40  0000 C CNN
-F 2 "" V 4980 2650 30  0000 C CNN
+F 2 "Resistors_SMD:R_0603_HandSoldering" V 4980 2650 30  0001 C CNN
 F 3 "" H 5050 2650 30  0000 C CNN
 	1    5050 2650
@@
 $EndComp
 $Comp
-L +3.3V #PWR058
+L +3.3V #PWR57
 U 1 1 55667746
 P 5050 2350
-F 0 "#PWR058" H 5050 2310 30  0001 C CNN
+F 0 "#PWR57" H 5050 2310 30  0001 C CNN
 F 1 "+3.3V" H 5050 2460 30  0000 C CNN
 F 2 "" H 5050 2350 60  0000 C CNN
@@
 $EndComp
 $Comp
-L GND #PWR059
+L GND #PWR58
 U 1 1 5566774C
 P 5900 3050
-F 0 "#PWR059" H 5900 3050 30  0001 C CNN
+F 0 "#PWR58" H 5900 3050 30  0001 C CNN
 F 1 "GND" H 5900 2980 30  0001 C CNN
 F 2 "" H 5900 3050 60  0000 C CNN
@@
 ESP8266 Wifi Module
 $Comp
-L +3.3V #PWR060
+L +3.3V #PWR63
 U 1 1 5566775A
 P 8000 4400
-F 0 "#PWR060" H 8000 4360 30  0001 C CNN
+F 0 "#PWR63" H 8000 4360 30  0001 C CNN
 F 1 "+3.3V" H 8000 4510 30  0000 C CNN
 F 2 "" H 8000 4400 60  0000 C CNN
@@
 $EndComp
 $Comp
-L +3.3V #PWR061
+L +3.3V #PWR56
 U 1 1 55667760
 P 4150 3950
-F 0 "#PWR061" H 4150 3910 30  0001 C CNN
+F 0 "#PWR56" H 4150 3910 30  0001 C CNN
 F 1 "+3.3V" H 4150 4060 30  0000 C CNN
 F 2 "" H 4150 3950 60  0000 C CNN
@@
 $EndComp
 $Comp
-L GND #PWR062
+L GND #PWR62
 U 1 1 5566776E
 P 7500 5350
-F 0 "#PWR062" H 7500 5350 30  0001 C CNN
+F 0 "#PWR62" H 7500 5350 30  0001 C CNN
 F 1 "GND" H 7500 5280 30  0001 C CNN
 F 2 "" H 7500 5350 60  0000 C CNN
@@
 F 0 "R11" V 7580 4900 40  0000 C CNN
 F 1 "R" V 7507 4901 40  0000 C CNN
-F 2 "" V 7430 4900 30  0000 C CNN
+F 2 "Resistors_SMD:R_0603_HandSoldering" V 7430 4900 30  0001 C CNN
 F 3 "" H 7500 4900 30  0000 C CNN
 	1    7500 4900
@@
 $EndComp
 $Comp
-L +3.3V #PWR063
+L +3.3V #PWR54
 U 1 1 5566915C
 P 2750 4500
-F 0 "#PWR063" H 2750 4460 30  0001 C CNN
+F 0 "#PWR54" H 2750 4460 30  0001 C CNN
 F 1 "+3.3V" H 2750 4610 30  0000 C CNN
 F 2 "" H 2750 4500 60  0000 C CNN
@@
 $EndComp
 $Comp
-L GND #PWR064
+L GND #PWR61
 U 1 1 556691BF
 P 7250 5000
-F 0 "#PWR064" H 7250 5000 30  0001 C CNN
+F 0 "#PWR61" H 7250 5000 30  0001 C CNN
 F 1 "GND" H 7250 4930 30  0001 C CNN
 F 2 "" H 7250 5000 60  0000 C CNN
@@
 F 0 "C12" H 3450 4950 40  0000 L CNN
 F 1 "C" H 3456 4765 40  0000 L CNN
-F 2 "" H 3488 4700 30  0000 C CNN
+F 2 "Capacitors_SMD:C_0603_HandSoldering" H 3488 4700 30  0001 C CNN
 F 3 "" H 3450 4850 60  0000 C CNN
 	1    3450 4850
@@
 $EndComp
 $Comp
-L GND #PWR065
+L GND #PWR55
 U 1 1 5566925F
 P 3450 5150
-F 0 "#PWR065" H 3450 5150 30  0001 C CNN
+F 0 "#PWR55" H 3450 5150 30  0001 C CNN
 F 1 "GND" H 3450 5080 30  0001 C CNN
 F 2 "" H 3450 5150 60  0000 C CNN
@@
 F 0 "TP2" H 1200 6050 60  0000 C CNN
 F 1 "TESTPOINT" H 1200 5750 60  0001 C CNN
-F 2 "" H 1200 5800 60  0000 C CNN
+F 2 "Connect:PINTST" H 1200 5800 60  0001 C CNN
 F 3 "" H 1200 5800 60  0000 C CNN
 	1    1200 5800
@@
 F 0 "TP3" H 1200 6250 60  0000 C CNN
 F 1 "TESTPOINT" H 1200 5950 60  0001 C CNN
-F 2 "" H 1200 6000 60  0000 C CNN
+F 2 "Connect:PINTST" H 1200 6000 60  0001 C CNN
 F 3 "" H 1200 6000 60  0000 C CNN
 	1    1200 6000
@@
 F 0 "TP4" H 1200 6450 60  0000 C CNN
 F 1 "TESTPOINT" H 1200 6150 60  0001 C CNN
-F 2 "" H 1200 6200 60  0000 C CNN
+F 2 "Connect:PINTST" H 1200 6200 60  0001 C CNN
 F 3 "" H 1200 6200 60  0000 C CNN
 	1    1200 6200
@@
 F 0 "TP5" H 1200 6650 60  0000 C CNN
 F 1 "TESTPOINT" H 1200 6350 60  0001 C CNN
-F 2 "" H 1200 6400 60  0000 C CNN
+F 2 "Connect:PINTST" H 1200 6400 60  0001 C CNN
 F 3 "" H 1200 6400 60  0000 C CNN
 	1    1200 6400
@@
 F 0 "TP6" H 1200 6850 60  0000 C CNN
 F 1 "TESTPOINT" H 1200 6550 60  0001 C CNN
-F 2 "" H 1200 6600 60  0000 C CNN
+F 2 "Connect:PINTST" H 1200 6600 60  0001 C CNN
 F 3 "" H 1200 6600 60  0000 C CNN
 	1    1200 6600
@@
 F 0 "TP7" H 1200 7050 60  0000 C CNN
 F 1 "TESTPOINT" H 1200 6750 60  0001 C CNN
-F 2 "" H 1200 6800 60  0000 C CNN
+F 2 "Connect:PINTST" H 1200 6800 60  0001 C CNN
 F 3 "" H 1200 6800 60  0000 C CNN
 	1    1200 6800
@@
 F 0 "TP8" H 1200 7250 60  0000 C CNN
 F 1 "TESTPOINT" H 1200 6950 60  0001 C CNN
-F 2 "" H 1200 7000 60  0000 C CNN
+F 2 "Connect:PINTST" H 1200 7000 60  0001 C CNN
 F 3 "" H 1200 7000 60  0000 C CNN
 	1    1200 7000
@@
 F 0 "TP9" H 1200 7450 60  0000 C CNN
 F 1 "TESTPOINT" H 1200 7150 60  0001 C CNN
-F 2 "" H 1200 7200 60  0000 C CNN
+F 2 "Connect:PINTST" H 1200 7200 60  0001 C CNN
 F 3 "" H 1200 7200 60  0000 C CNN
 	1    1200 7200
@@
 F 0 "TP10" H 1200 7650 60  0000 C CNN
 F 1 "TESTPOINT" H 1200 7350 60  0001 C CNN
-F 2 "" H 1200 7400 60  0000 C CNN
+F 2 "Connect:PINTST" H 1200 7400 60  0001 C CNN
 F 3 "" H 1200 7400 60  0000 C CNN
 	1    1200 7400

Commit message: Remove Barrel Jack and associated power circuits. Unnecessary for now and add a lot of complexity / BOM cost
Parts:
- removed TP2, TP3, TP4, TP5, TP6, TP7, TP8: TESTPOINT, Connect:PINTST, symbol TESTPOINT
- P5: value CONN_4 -> ESP_PROG
Changed lines of the file:
@@
 P 6800 2350
 F 0 "P5" V 6750 2350 50  0000 C CNN
-F 1 "CONN_4" V 6850 2350 50  0000 C CNN
+F 1 "ESP_PROG" V 6850 2350 50  0000 C CNN
 F 2 "Pin_Headers:Pin_Header_Straight_1x04" H 6800 2350 60  0001 C CNN
 F 3 "" H 6800 2350 60  0000 C CNN
@@
 Text HLabel 4550 4200 0    39   Input ~ 0
 ESP_GPIO_16
-$Comp
-L TESTPOINT TP2
-U 1 1 55669763
-P 1200 5800
-F 0 "TP2" H 1200 6050 60  0000 C CNN
-F 1 "TESTPOINT" H 1200 5750 60  0001 C CNN
-F 2 "Connect:PINTST" H 1200 5800 60  0001 C CNN
-F 3 "" H 1200 5800 60  0000 C CNN
-	1    1200 5800
-	0    -1   -1   0
-$EndComp
 Wire Wire Line
 	6650 2700 6650 2900
@@
 Wire Wire Line
 	4850 4500 4550 4500
-$Comp
-L TESTPOINT TP3
-U 1 1 55669E4F
-P 1200 6000
-F 0 "TP3" H 1200 6250 60  0000 C CNN
-F 1 "TESTPOINT" H 1200 5950 60  0001 C CNN
-F 2 "Connect:PINTST" H 1200 6000 60  0001 C CNN
-F 3 "" H 1200 6000 60  0000 C CNN
-	1    1200 6000
-	0    -1   -1   0
-$EndComp
-$Comp
-L TESTPOINT TP4
-U 1 1 55669E83
-P 1200 6200
-F 0 "TP4" H 1200 6450 60  0000 C CNN
-F 1 "TESTPOINT" H 1200 6150 60  0001 C CNN
-F 2 "Connect:PINTST" H 1200 6200 60  0001 C CNN
-F 3 "" H 1200 6200 60  0000 C CNN
-	1    1200 6200
-	0    -1   -1   0
-$EndComp
-$Comp
-L TESTPOINT TP5
-U 1 1 55669EAD
-P 1200 6400
-F 0 "TP5" H 1200 6650 60  0000 C CNN
-F 1 "TESTPOINT" H 1200 6350 60  0001 C CNN
-F 2 "Connect:PINTST" H 1200 6400 60  0001 C CNN
-F 3 "" H 1200 6400 60  0000 C CNN
-	1    1200 6400
-	0    -1   -1   0
-$EndComp
-$Comp
-L TESTPOINT TP6
-U 1 1 55669F01
-P 1200 6600
-F 0 "TP6" H 1200 6850 60  0000 C CNN
-F 1 "TESTPOINT" H 1200 6550 60  0001 C CNN
-F 2 "Connect:PINTST" H 1200 6600 60  0001 C CNN
-F 3 "" H 1200 6600 60  0000 C CNN
-	1    1200 6600
-	0    -1   -1   0
-$EndComp
-$Comp
-L TESTPOINT TP7
-U 1 1 55669F33
-P 1200 6800
-F 0 "TP7" H 1200 7050 60  0000 C CNN
-F 1 "TESTPOINT" H 1200 6750 60  0001 C CNN
-F 2 "Connect:PINTST" H 1200 6800 60  0001 C CNN
-F 3 "" H 1200 6800 60  0000 C CNN
-	1    1200 6800
-	0    -1   -1   0
-$EndComp
-$Comp
-L TESTPOINT TP8
-U 1 1 55669F6B
-P 1200 7000
-F 0 "TP8" H 1200 7250 60  0000 C CNN
-F 1 "TESTPOINT" H 1200 6950 60  0001 C CNN
-F 2 "Connect:PINTST" H 1200 7000 60  0001 C CNN
-F 3 "" H 1200 7000 60  0000 C CNN
-	1    1200 7000
-	0    -1   -1   0
-$EndComp
-Wire Wire Line
-	1200 5800 1600 5800
-Wire Wire Line
-	1200 6000 1600 6000
-Wire Wire Line
-	1200 6200 1600 6200
-Wire Wire Line
-	1200 6400 1600 6400
-Wire Wire Line
-	1200 6600 1600 6600
-Wire Wire Line
-	1200 6800 1600 6800
-Wire Wire Line
-	1200 7000 1600 7000
-Text HLabel 1600 5800 2    39   Input ~ 0
-ESP_GPIO_16
-Text HLabel 1600 6200 2    39   Input ~ 0
-ESP_GPIO_5
-Text HLabel 1600 6000 2    39   Input ~ 0
-ESP_GPIO_4
 $Comp
 L TESTPOINT TP9
@@
 Wire Notes Line
 	600  7700 600  5500
-Text Notes 1300 5650 0    60   ~ 0
+Text Notes 1250 6900 0    60   ~ 0
 Test Points
 Text HLabel 4650 3900 0    39   Input ~ 0
@@
 Text HLabel 8000 4500 2    39   Input ~ 0
 ESP_GPIO_15
-Text HLabel 1600 6400 2    39   Input ~ 0
-ESP_GPIO_15
-Text HLabel 1600 6600 2    39   Input ~ 0
-ESP_GPIO_12
-Text HLabel 1600 6800 2    39   Input ~ 0
-ESP_GPIO_14
-Text HLabel 1600 7000 2    39   Input ~ 0
-ESP_GPIO_13
 Wire Wire Line
 	7250 3900 8000 3900
